Commit message: rename overhead camera stand to overhead_camera
Prefix every stand link/joint and the D435i sensor with overhead_camera so
the overhead camera can coexist with the follower variant's wrist D405,
which is named camera.

Co-Authored-By: Claude Opus 5.5 <noreply@anthropic.com>

File: urdf/macros/camera_with_stand.xacro (robot description, xacro)
@@ -14,9 +14,10 @@
             <xacro:include filename="$(find realsense2_description)/urdf/_d435i.urdf.xacro"/>
         </xacro:if>
-        <!-- Links -->
-        <link name="camera_mount_link"/>
-        <link name="camera_base_link"/>
+        <!-- Links (all stand and sensor names carry the 'overhead_camera' prefix so that they do
+             not clash with the follower variant's wrist D405, which is named 'camera') -->
+        <link name="overhead_camera_mount_link"/>
+        <link name="overhead_camera_base_link"/>
         <xacro:if value="${camera_type != 'realsense'}">
-            <link name="camera_link">
+            <link name="overhead_camera_link">
                 <visual>
                     <origin xyz="0 0 -0.015" rpy="0 0 0"/>
@@ -28,5 +29,5 @@
             </link>
         </xacro:if>
-        <link name="camera_holder_upper_arm_link">
+        <link name="overhead_camera_holder_upper_arm_link">
             <visual>
                 <origin xyz="0.015 0 -0.15" rpy="0 0 0"/>
@@ -43,5 +44,5 @@
             </collision>
         </link>
-        <link name="camera_holder_lower_arm_link">
+        <link name="overhead_camera_holder_lower_arm_link">
             <visual>
                 <origin xyz="${camera_pos_z/2} 0 0.015" rpy="0 0 0"/>
@@ -58,5 +59,5 @@
             </collision>
         </link>
-        <link name="camera_holder_base">
+        <link name="overhead_camera_holder_base">
             <visual>
                 <geometry>
@@ -68,34 +69,34 @@
         </link>
         <!-- Joints -->
-        <joint name="camera_mount_camera_base_joint" type="fixed">
-            <parent link="camera_mount_link"/>
-            <child link="camera_base_link"/>
+        <joint name="overhead_camera_mount_camera_base_joint" type="fixed">
+            <parent link="overhead_camera_mount_link"/>
+            <child link="overhead_camera_base_link"/>
             <origin xyz="0 0 0" rpy="${camera_roll} ${camera_pitch} ${camera_yaw}"/>
         </joint>
         <xacro:if value="${camera_type == 'realsense'}">
-            <xacro:sensor_d435i parent="camera_base_link" use_nominal_extrinsics="true" >
+            <xacro:sensor_d435i name="overhead_camera" parent="overhead_camera_base_link" use_nominal_extrinsics="true" >
                 <origin xyz="0.0095 0 -0.0125" rpy="0 0 0"/>
             </xacro:sensor_d435i>
         </xacro:if>
         <xacro:if value="${camera_type != 'realsense'}">
-            <joint name="camera_base_to_camera_joint" type="fixed">
-                <parent link="camera_base_link"/>
-                <child link="camera_link"/>
+            <joint name="overhead_camera_base_to_camera_joint" type="fixed">
+                <parent link="overhead_camera_base_link"/>
+                <child link="overhead_camera_link"/>
                 <origin xyz="0 0 0" rpy="0 ${pi_val/2} 0"/>
             </joint>
         </xacro:if>
-        <joint name="camera_base_to_upper_arm_joint" type="fixed">
-            <parent link="camera_mount_link"/>
-            <child link="camera_holder_upper_arm_link"/>
+        <joint name="overhead_camera_base_to_upper_arm_joint" type="fixed">
+            <parent link="overhead_camera_mount_link"/>
+            <child link="overhead_camera_holder_upper_arm_link"/>
             <origin xyz="-0.0125 0 0.03" rpy="${pi_val} ${pi_val/2} 0"/>
         </joint>
-        <joint name="camera_holder_upper_arm_to_camera_holder_lower_arm_joint" type="fixed">
-            <parent link="camera_holder_upper_arm_link"/>
-            <child link="camera_holder_lower_arm_link"/>
+        <joint name="overhead_camera_holder_upper_arm_to_camera_holder_lower_arm_joint" type="fixed">
+            <parent link="overhead_camera_holder_upper_arm_link"/>
+            <child link="overhead_camera_holder_lower_arm_link"/>
             <origin xyz="0.03 0 -0.3" rpy="0 0 0"/>
         </joint>
-        <joint name="camera_holder_lower_arm_to_camera_holder_base_joint" type="fixed">
-            <parent link="camera_holder_lower_arm_link"/>
-            <child link="camera_holder_base"/>
+        <joint name="overhead_camera_holder_lower_arm_to_camera_holder_base_joint" type="fixed">
+            <parent link="overhead_camera_holder_lower_arm_link"/>
+            <child link="overhead_camera_holder_base"/>
             <origin xyz="${camera_pos_z} 0 0.015" rpy="0 ${pi_val/2} 0"/>
         </joint>

File: urdf/wxai.urdf.xacro (robot description, xacro)
@@ -45,8 +45,10 @@
                                 camera_roll="$(arg camera_pos_roll)" camera_pitch="$(arg camera_pos_pitch)" camera_yaw="$(arg camera_pos_yaw)"
                                 camera_type="$(arg camera_type)" />
-      <!-- Connect camera to robot base -->
-      <joint name="$(arg prefix)base_link_camera_mount_joint" type="fixed">
+      <!-- Connect the overhead camera stand to the robot base. Its links/frames use the
+           'overhead_camera' prefix so they can coexist with the follower variant's wrist
+           D405 ('<prefix>camera_*'). They are not arm-prefixed: there is one stand per scene. -->
+      <joint name="$(arg prefix)base_link_overhead_camera_mount_joint" type="fixed">
           <parent link="$(arg prefix)base_link"/>
-          <child link="camera_mount_link"/>
+          <child link="overhead_camera_mount_link"/>
           <origin xyz="$(arg camera_pos_x) $(arg camera_pos_y) $(arg camera_pos_z)"
                   rpy="$(arg camera_holder_roll) $(arg camera_holder_pitch) $(arg camera_holder_yaw)"/>
